Commit message: simulation: lidar ok

File: src/utcrobot23/description/gazebo_control.xacro (robot description, xacro)
@@ -6,9 +6,9 @@
             <left_joint>left_wheel_joint</left_joint>
             <right_joint>right_wheel_joint</right_joint>
-            <wheel_separation>0.35</wheel_separation>
-            <wheel_diameter>0.1</wheel_diameter>
+            <wheel_separation>0.2032</wheel_separation>
+            <wheel_diameter>0.034</wheel_diameter>
             <!-- Limits -->
             <max_wheel_torque>200</max_wheel_torque>
-            <max_wheel_acceleration>10.0</max_wheel_acceleration>
+            <max_wheel_acceleration>5.0</max_wheel_acceleration>
             <!-- Output -->
             <odometry_frame>odom</odometry_frame>

File: src/utcrobot23/description/lidar.xacro (robot description, xacro)
@@ -18,6 +18,6 @@
             </geometry>
         </collision>
-        <xacro:inertial_box mass="0.16" x="0.05" y="0.05" z="0.070">
-            <origin xyz="0 0 0" rpy="0 0 0"/>
+        <xacro:inertial_box mass="0.1" x="0.05" y="0.05" z="0.070">
+            <origin xyz="0.03 0 0.065" rpy="0 0 0"/>
         </xacro:inertial_box>
     </link>

File: src/utcrobot23/description/robot.urdf.xacro (robot description, xacro)
@@ -1,7 +1,12 @@
 <?xml version="1.0"?>
 <robot xmlns:xacro="http://www.ros.org/wiki/xacro"  name="robot">
-     <!--<xacro:include filename="ros2_control.xacro" />-->
+    <xacro:arg name="use_ros2_control" default="true"/>
     <xacro:include filename="robot_core.xacro" />
-    <xacro:include filename="gazebo_control.xacro"/>
+    <xacro:if value="$(arg use_ros2_control)">
+        <xacro:include filename="ros2_control.xacro" />
+    </xacro:if>
+    <xacro:unless value="$(arg use_ros2_control)">
+       <xacro:include filename="gazebo_control.xacro"/>
+    </xacro:unless>
     <xacro:include filename="lidar.xacro"/>
 </robot>

File: src/utcrobot23/description/robot_core.xacro (robot description, xacro)
@@ -63,5 +63,5 @@
         <collision>
             <geometry>
-                <cylinder radius="0.034" length="0.0254"/>
+                <sphere radius="0.034"/>
             </geometry>
         </collision>
@@ -89,5 +89,5 @@
         <collision>
             <geometry>
-                <cylinder radius="0.034" length="0.0254"/>
+                <sphere radius="0.034"/>
             </geometry>
         </collision>
@@ -126,3 +126,30 @@
         <mu2 value="0.001"/>
     </gazebo>
+        <!--  CASTER WHEEL LINK
+    <joint name="caster_wheel_joint2" type="fixed">
+        <parent link="chassis"/>
+        <child link="caster_wheel2"/>
+        <origin xyz="0.1 0 -0.023"/>
+    </joint>
+    <link name="caster_wheel2">
+        <visual>
+            <geometry>
+                <sphere radius="0.007"/>
+            </geometry>
+            <material name="black"/>
+        </visual>
+        <collision>
+            <geometry>
+                <sphere radius="0.007"/>
+            </geometry>
+        </collision>
+        <xacro:inertial_sphere mass="0.01" radius="0.007">
+            <origin xyz="0.1 0 -0.023" rpy="0 0 0"/>
+        </xacro:inertial_sphere>
+    </link>
+    <gazebo reference="caster_wheel2">
+        <material>Gazebo/Black</material>
+        <mu1 value="0.001"/>
+        <mu2 value="0.001"/>
+    </gazebo>-->
 </robot>

File: src/utcrobot23/description/ros2_control.xacro (robot description, xacro)
@@ -22,8 +22,8 @@
         </joint>
     </ros2_control>
-    <!--<gazebo>
+    <gazebo>
         <plugin name="gazebo_ros2_control" filename="libgazebo_ros2_control.so">
             <parameters>$(find utcrobot23)/config/my_controllers.yaml</parameters>
         </plugin>
-    </gazebo>-->
+    </gazebo>-
 </robot>

Commit message: resolution problème inertie

File: src/utcrobot23/description/gazebo_control.xacro (robot description, xacro)
@@ -9,6 +9,6 @@
             <wheel_diameter>0.034</wheel_diameter>
             <!-- Limits -->
-            <max_wheel_torque>200</max_wheel_torque>
-            <max_wheel_acceleration>5.0</max_wheel_acceleration>
+            <max_wheel_torque>0.00005</max_wheel_torque>
+            <max_wheel_acceleration>0.00003</max_wheel_acceleration>
             <!-- Output -->
             <odometry_frame>odom</odometry_frame>

File: src/utcrobot23/description/lidar.xacro (robot description, xacro)
@@ -19,5 +19,5 @@
         </collision>
         <xacro:inertial_box mass="0.1" x="0.05" y="0.05" z="0.070">
-            <origin xyz="0.03 0 0.065" rpy="0 0 0"/>
+            <origin xyz="0 0 0" rpy="0 0 0"/>
         </xacro:inertial_box>
     </link>

File: src/utcrobot23/description/robot_core.xacro (robot description, xacro)
@@ -20,4 +20,12 @@
     <link name="base_link">
     </link>
+    <!-- BASE_FOOTPRINT LINK -->
+    <joint name="base_footprint_joint" type="fixed">
+        <parent link="base_link"/>
+        <child link="base_footprint"/>
+        <origin xyz="0 0 0" rpy="0 0 0"/>
+    </joint>
+    <link name="base_footprint">
+    </link>
     <!--  CHASSIS LINK  -->
     <joint name="chassis_joint" type="fixed">
@@ -37,9 +45,9 @@
             <origin xyz="0 0 0.007"/>
             <geometry>
-                <box size="0.140 0.320 0.0455"/>
+                <box size="0.140 0.200 0.0455"/>
             </geometry>
         </collision>
         <xacro:inertial_box mass="0.5" x="0.140" y="0.320" z="0.0455">
-            <origin xyz="0.0 0.0 0.007" rpy="0 0 0"/>
+            <origin xyz="0 0 0" rpy="0 0 0"/>
         </xacro:inertial_box>
     </link>
@@ -67,5 +75,5 @@
         </collision>
         <xacro:inertial_sphere mass="0.1" radius="0.034" >
-            <origin xyz="0 0.1016 0.0425" rpy="0 0 0"/>
+            <origin xyz="0 0 0" rpy="0 0 0"/>
         </xacro:inertial_sphere>
     </link>
@@ -93,5 +101,5 @@
         </collision>
         <xacro:inertial_sphere mass="0.1" radius="0.034" >
-            <origin xyz="0 -0.1016 0.00425" rpy="0 0 0"/>
+            <origin xyz="0 0 0" rpy="0 0 0"/>
         </xacro:inertial_sphere>
     </link>
@@ -118,17 +126,17 @@
         </collision>
         <xacro:inertial_sphere mass="0.01" radius="0.007">
-            <origin xyz="0.05 0 -0.023" rpy="0 0 0"/>
+            <origin xyz="0 0 0" rpy="0 0 0"/>
         </xacro:inertial_sphere>
     </link>
     <gazebo reference="caster_wheel">
         <material>Gazebo/Black</material>
-        <mu1 value="0.05"/>
-        <mu2 value="0.05"/>
+        <mu1 value="0.0"/>
+        <mu2 value="0.0"/>
     </gazebo>
-        <!--  CASTER WHEEL LINK
+        <!--  CASTER WHEEL LINK >
     <joint name="caster_wheel_joint2" type="fixed">
         <parent link="chassis"/>
         <child link="caster_wheel2"/>
-        <origin xyz="0.1 0 -0.023"/>
+        <origin xyz="-0.05 0 -0.023"/>
     </joint>
     <link name="caster_wheel2">
@@ -150,6 +158,6 @@
     <gazebo reference="caster_wheel2">
         <material>Gazebo/Black</material>
-        <mu1 value="0.001"/>
-        <mu2 value="0.001"/>
-    </gazebo>-->
+        <mu1 value="0.0"/>
+        <mu2 value="0.0"/>
+    </gazebo-->
 </robot>

Commit message: slam

File: src/utcrobot23/description/gazebo_control.xacro (robot description, xacro)
@@ -6,6 +6,6 @@
             <left_joint>left_wheel_joint</left_joint>
             <right_joint>right_wheel_joint</right_joint>
-            <wheel_separation>0.2032</wheel_separation>
-            <wheel_diameter>0.034</wheel_diameter>
+            <wheel_separation>0.3085</wheel_separation>
+            <wheel_diameter>0.035</wheel_diameter>
             <!-- Limits -->
             <max_wheel_torque>0.00005</max_wheel_torque>

File: src/utcrobot23/description/lidar.xacro (robot description, xacro)
@@ -4,5 +4,5 @@
         <parent link="chassis"/>
         <child link="laser_frame"/>
-        <origin xyz="0.03 0 0.065" rpy="0 0 ${pi}"/>
+        <origin xyz="0.03 0 0.06" rpy="0 0 ${pi}"/>
     </joint>
     <link name="laser_frame">
@@ -31,5 +31,5 @@
                 <scan>
                     <horizontal>
-                        <samples>240</samples>
+                        <samples>1000</samples>
                         <resolution>0.36</resolution>
                         <min_angle>-3.14</min_angle>

File: src/utcrobot23/description/robot_core.xacro (robot description, xacro)
@@ -59,5 +59,5 @@
         <parent link="chassis"/>
         <child link="left_wheel"/>
-        <origin xyz="0 0.1016 0.00425" rpy="-${pi/2} 0 0"/>
+        <origin xyz="0 0.15425 0" rpy="-${pi/2} 0 0"/>
         <axis xyz="0 0 1"/>
     </joint>
@@ -65,5 +65,5 @@
         <visual>
             <geometry>
-                <cylinder radius="0.034" length="0.0254"/>
+                <cylinder radius="0.035" length="0.0254"/>
             </geometry>
             <material name="blue"/>
@@ -71,8 +71,8 @@
         <collision>
             <geometry>
-                <sphere radius="0.034"/>
+                <sphere radius="0.035"/>
             </geometry>
         </collision>
-        <xacro:inertial_sphere mass="0.1" radius="0.034" >
+        <xacro:inertial_sphere mass="0.1" radius="0.035" >
             <origin xyz="0 0 0" rpy="0 0 0"/>
         </xacro:inertial_sphere>
@@ -85,5 +85,5 @@
         <parent link="chassis"/>
         <child link="right_wheel"/>
-        <origin xyz="0 -0.1016 0.00425" rpy="${pi/2} 0 0"/>
+        <origin xyz="0 -0.15425 0" rpy="${pi/2} 0 0"/>
         <axis xyz="0 0 -1"/>
     </joint>
@@ -91,5 +91,5 @@
         <visual>
             <geometry>
-                <cylinder radius="0.034" length="0.0254"/>
+                <cylinder radius="0.035" length="0.0254"/>
             </geometry>
             <material name="blue"/>
@@ -97,8 +97,8 @@
         <collision>
             <geometry>
-                <sphere radius="0.034"/>
+                <sphere radius="0.035"/>
             </geometry>
         </collision>
-        <xacro:inertial_sphere mass="0.1" radius="0.034" >
+        <xacro:inertial_sphere mass="0.1" radius="0.035" >
             <origin xyz="0 0 0" rpy="0 0 0"/>
         </xacro:inertial_sphere>
@@ -111,10 +111,10 @@
         <parent link="chassis"/>
         <child link="caster_wheel"/>
-        <origin xyz="0.05 0 -0.023"/>
+        <origin xyz="0.05 0 -0.025"/>
     </joint>
     <link name="caster_wheel">
         <visual>
             <geometry>
-                <sphere radius="0.007"/>
+                <sphere radius="0.01"/>
             </geometry>
             <material name="black"/>
@@ -122,8 +122,8 @@
         <collision>
             <geometry>
-                <sphere radius="0.007"/>
+                <sphere radius="0.01"/>
             </geometry>
         </collision>
-        <xacro:inertial_sphere mass="0.01" radius="0.007">
+        <xacro:inertial_sphere mass="0.01" radius="0.01">
             <origin xyz="0 0 0" rpy="0 0 0"/>
         </xacro:inertial_sphere>
