Commit message: 2 lidars

File: src/utcrobot23/description/lidar_2nd.xacro (robot description, xacro)
@@ -1,10 +1,10 @@
 <?xml version="1.0"?>
 <robot xmlns:xacro="http://www.ros.org/wiki/xacro" >
-    <joint name= "laser_joint" type="fixed">
+    <joint name= "laser_joint2" type="fixed">
         <parent link="chassis"/>
-        <child link="laser_frame"/>
-        <origin xyz="0.03 0 0.06" rpy="0 ${pi} ${pi}"/>
+        <child link="laser_frame2"/>
+        <origin xyz="-0.03 0 0.06" rpy="0 0 ${pi}"/>
     </joint>
-    <link name="laser_frame">
+    <link name="laser_frame2">
          <visual>
             <geometry>
@@ -22,7 +22,7 @@
         </xacro:inertial_box>
     </link>
-    <gazebo reference="laser_frame">
+    <gazebo reference="laser_frame2">
         <material>Gazebo/Red</material>
-        <sensor name="laser" type="ray">
+        <sensor name="laser2" type="ray">
             <pose> 0 0 0 0 0 0 </pose>
             <visualize>true</visualize>
@@ -43,10 +43,10 @@
                 </range>
             </ray>
-            <plugin name="laser_controller" filename="libgazebo_ros_ray_sensor.so">
+            <plugin name="laser_controller2" filename="libgazebo_ros_ray_sensor.so">
                 <ros>
                     <argument>~/out:=scan</argument>
                 </ros>
                 <output_type>sensor_msgs/LaserScan</output_type>
-                <frame_name>laser_frame</frame_name>
+                <frame_name>laser_frame2</frame_name>
             </plugin>
         </sensor>

File: src/utcrobot23/description/robot.urdf.xacro (robot description, xacro)
@@ -11,3 +11,4 @@
     </xacro:unless>
     <xacro:include filename="lidar.xacro"/>
+    <xacro:include filename="lidar_2nd.xacro"/>
 </robot>

Commit message: rotation 2nd lidar

File: src/utcrobot23/description/lidar_2nd.xacro (robot description, xacro)
@@ -4,5 +4,5 @@
         <parent link="chassis"/>
         <child link="laser_frame2"/>
-        <origin xyz="-0.03 0 0.06" rpy="0 0 ${pi}"/>
+        <origin xyz="-0.03 0 0.06" rpy="${pi} 0 ${pi}"/>
     </joint>
     <link name="laser_frame2">
