Commit message: test changement de base

File: src/utcrobot23/description/lidar.xacro (robot description, xacro)
@@ -4,5 +4,5 @@
         <parent link="chassis"/>
         <child link="laser_frame"/>
-        <origin xyz="0.03 0 0.065" rpy="${pi} 0 ${pi}"/>
+        <origin xyz="0.03 0 0.065" rpy="0 0 ${pi}"/>
     </joint>
     <link name="laser_frame">

Commit message: test base lidar

File: src/utcrobot23/description/lidar.xacro (robot description, xacro)
@@ -4,5 +4,5 @@
         <parent link="chassis"/>
         <child link="laser_frame"/>
-        <origin xyz="0.03 0 0.06" rpy="0 0 ${pi}"/>
+        <origin xyz="0.03 0 0.06" rpy="0 ${pi} ${pi}"/>
     </joint>
     <link name="laser_frame">

Commit message: lidar changement position

File: src/utcrobot23/description/lidar.xacro (robot description, xacro)
@@ -4,5 +4,6 @@
         <parent link="chassis"/>
         <child link="laser_frame"/>
-        <origin xyz="0.03 0 0.06" rpy="0 ${pi} ${pi}"/>
+        <origin xyz="0.0 -0.19 0.0" rpy="${pi} 0 ${-pi/2}"/>
+        <!-- <origin xyz="0.03 0 0.06" rpy="0 ${pi} ${pi}"/> -->
     </joint>
     <link name="laser_frame">
@@ -31,8 +32,8 @@
                 <scan>
                     <horizontal>
-                        <samples>318</samples>
+                        <samples>636</samples>
                         <resolution>0.36</resolution>
-                        <min_angle>-1.00</min_angle>
-                        <max_angle>1.00</max_angle>
+                        <min_angle>-2.0</min_angle>
+                        <max_angle>2.0</max_angle>
                     </horizontal>
                 </scan>

File: src/utcrobot23/description/lidar_2nd.xacro (robot description, xacro)
@@ -4,5 +4,6 @@
         <parent link="chassis"/>
         <child link="laser_frame2"/>
-        <origin xyz="-0.03 0 0.06" rpy="${pi} 0 ${pi}"/>
+        <origin xyz="0.0 0.19 0.0" rpy="${pi} 0 ${pi/2}"/>
+        <!-- <origin xyz="-0.03 0 0.06" rpy="${pi} 0 ${pi}"/> -->
     </joint>
     <link name="laser_frame2">
@@ -31,8 +32,8 @@
                 <scan>
                     <horizontal>
-                        <samples>318</samples>
+                        <samples>636</samples>
                         <resolution>0.36</resolution>
-                        <min_angle>-1.00</min_angle>
-                        <max_angle>1.00</max_angle>
+                        <min_angle>-2.0</min_angle>
+                        <max_angle>2.0</max_angle>
                     </horizontal>
                 </scan>

File: src/utcrobot23/description/robot_core.xacro (robot description, xacro)
@@ -45,4 +45,22 @@
             <origin xyz="0 0 0.007"/>
             <geometry>
+                <box size="0.140 0.320 0.0455"/>
+            </geometry>
+        </collision>
+        <xacro:inertial_box mass="0.5" x="0.140" y="0.320" z="0.0455">
+            <origin xyz="0 0 0" rpy="0 0 0"/>
+        </xacro:inertial_box>
+    </link>
+    <!-- <link name="chassis">
+        <visual>
+            <origin xyz="0 0 0.007"/>
+            <geometry>
+                <box size="0.140 0.320 0.0455"/>
+            </geometry>
+            <material name="white"/>
+        </visual>
+        <collision>
+            <origin xyz="0 0 0.007"/>
+            <geometry>
                 <box size="0.140 0.200 0.0455"/>
             </geometry>
@@ -51,5 +69,5 @@
             <origin xyz="0 0 0" rpy="0 0 0"/>
         </xacro:inertial_box>
-    </link>
+    </link> -->
     <gazebo reference="chassis">
         <material>Gazebo/White</material>
