Commit message: arrangement sim presque parfait

File: src/utcrobot23/description/robot_core.xacro (robot description, xacro)
@@ -41,5 +41,5 @@
         </collision>
         <xacro:inertial_box mass="0.5" x="0.140" y="0.320" z="0.0455">
-            <origin xyz="0.004 0.001 0.051" rpy="0 0 0"/>
+            <origin xyz="0.0 0.0 0.007" rpy="0 0 0"/>
         </xacro:inertial_box>
     </link>
@@ -66,7 +66,7 @@
             </geometry>
         </collision>
-        <xacro:inertial_cylinder mass="0.1" length="0.0254" radius="0.034">
-            <origin xyz="0 0 0.0425" rpy="0 0 0"/>
-        </xacro:inertial_cylinder>
+        <xacro:inertial_sphere mass="0.1" radius="0.034" >
+            <origin xyz="0 0.1016 0.0425" rpy="0 0 0"/>
+        </xacro:inertial_sphere>
     </link>
     <gazebo reference="left_wheel">
@@ -92,7 +92,7 @@
             </geometry>
         </collision>
-        <xacro:inertial_cylinder mass="0.1" length="0.0254" radius="0.034">
-            <origin xyz="0 0 0.00425" rpy="0 0 0"/>
-        </xacro:inertial_cylinder>
+        <xacro:inertial_sphere mass="0.1" radius="0.034" >
+            <origin xyz="0 -0.1016 0.00425" rpy="0 0 0"/>
+        </xacro:inertial_sphere>
     </link>
     <gazebo reference="right_wheel">
@@ -123,6 +123,6 @@
     <gazebo reference="caster_wheel">
         <material>Gazebo/Black</material>
-        <mu1 value="0.001"/>
-        <mu2 value="0.001"/>
+        <mu1 value="0.05"/>
+        <mu2 value="0.05"/>
     </gazebo>
         <!--  CASTER WHEEL LINK

Commit message: move_to_pose

File: src/utcrobot23/description/robot_core.xacro (robot description, xacro)
@@ -75,5 +75,5 @@
     <!--  LEFT WHEEL LINK  -->
     <joint name="left_wheel_joint" type="continuous">
-        <parent link="chassis"/>
+        <parent link="base_link"/>
         <child link="left_wheel"/>
         <origin xyz="0 0.15425 0" rpy="-${pi/2} 0 0"/>
@@ -101,5 +101,5 @@
     <!--  RIGHT WHEEL LINK  -->
     <joint name="right_wheel_joint" type="continuous">
-        <parent link="chassis"/>
+        <parent link="base_link"/>
         <child link="right_wheel"/>
         <origin xyz="0 -0.15425 0" rpy="${pi/2} 0 0"/>
@@ -127,5 +127,5 @@
     <!--  CASTER WHEEL LINK-->
     <joint name="caster_wheel_joint" type="fixed">
-        <parent link="chassis"/>
+        <parent link="base_link"/>
         <child link="caster_wheel"/>
         <origin xyz="0.05 0 -0.025"/>
